File: adjustableBuck.kicad_pcb (KiCad board)
At the start: 2 copper layers, 75 parts, among them Q1 IPB048N15N5LF, Q2 IPB048N15N5LF, Q3 IPB048N15N5LF, Q4 IPB048N15N5LF, Q5 IPB048N15N5LF, Q6 BC547, SW1 DIP6, SW2 DIP2, SW3 DIP6, SW4 76SD01ST, SW5 DIP6, U1 LT8210EFE

Commit message: First board layout
Parts:
- removed C2: 470uF 35V, PCM_Capacitor_THT_AKL:CP_Radial_D10.0mm_P5.00mm
- removed C3: 10uF 100V, Capacitor_SMD:C_1210_3225Metric_Pad1.33x2.70mm_HandSolder
- removed C6: C_0805, PCM_Capacitor_SMD_AKL:C_0805_2012Metric
- removed D1: MURS160, PCM_Diode_SMD_AKL:D_SMB
- removed R19: 10k, PCM_Resistor_SMD_AKL:R_0805_2012Metric_Pad1.20x1.40mm_HandSolder
- removed R3, R4: R_0805, PCM_Resistor_SMD_AKL:R_0805_2012Metric_Pad1.20x1.40mm_HandSolder
- removed SW1: DIP6, Button_Switch_SMD:6DIPCFS
- added C25: 4.7uF 35v, PCM_Capacitor_SMD_AKL:C_0805_2012Metric, F.Cu at (233.5, 55.8)
- added C26: 4.7uF 35v, PCM_Capacitor_SMD_AKL:C_0805_2012Metric, F.Cu at (233.5, 58.2)
- added R33: 10k, PCM_Resistor_SMD_AKL:R_0805_2012Metric_Pad1.20x1.40mm_HandSolder, F.Cu at (171.1, 118.1)
- added R34: 10k, PCM_Resistor_SMD_AKL:R_0805_2012Metric_Pad1.20x1.40mm_HandSolder, F.Cu at (173.7, 118.1)
- added SW6: DIP2, Button_Switch_SMD:2DIPCFS, F.Cu at (180.9, 110.7)
- added TP10: TestPoint, Connector_Pin:Pin_D1.3mm_L11.0mm, F.Cu at (158.5, 82.5)
- added TP11: TestPoint, Connector_Pin:Pin_D1.3mm_L11.0mm, F.Cu at (178.7, 72.5)
- added TP12: TestPoint, Connector_Pin:Pin_D1.3mm_L11.0mm, F.Cu at (158.5, 97.5)
- added TP13: TestPoint, Connector_Pin:Pin_D1.3mm_L11.0mm, F.Cu at (178.7, 87.5)
- added TP14: TestPoint, Connector_Pin:Pin_D1.3mm_L11.0mm, F.Cu at (178.7, 97.5)
- added TP15: TestPoint, Connector_Pin:Pin_D1.3mm_L11.0mm, F.Cu at (178.7, 92.7)
- added TP16: TestPoint, Connector_Pin:Pin_D1.3mm_L11.0mm, F.Cu at (158.5, 72.5)
- added TP18: TestPoint, Connector_Pin:Pin_D1.3mm_L11.0mm, F.Cu at (158.5, 77.5)
- added TP19: TestPoint, Connector_Pin:Pin_D1.3mm_L11.0mm, F.Cu at (158.5, 92.5)
- added TP2: TestPoint, Connector_Pin:Pin_D1.3mm_L11.0mm, F.Cu at (158.5, 87.5)
- added TP21: TestPoint, Connector_Pin:Pin_D1.3mm_L11.0mm, F.Cu at (234.0, 74.5)
- added TP4: ProbePoint, Connector_Pin:Pin_D1.1mm_L10.2mm_W3.5mm_Flat, F.Cu at (161.8, 44.5)
- added TP5: ProbePoint, Connector_Pin:Pin_D1.1mm_L10.2mm_W3.5mm_Flat, F.Cu at (242.0, 63.5)
- added TP6: ProbePoint, Connector_Pin:Pin_D1.1mm_L10.2mm_W3.5mm_Flat, F.Cu at (242.0, 74.5)
- added TP7: TestPoint, Connector_Pin:Pin_D1.3mm_L11.0mm, F.Cu at (169.5, 36.5)
- added TP8: TestPoint, Connector_Pin:Pin_D1.3mm_L11.0mm, F.Cu at (234.0, 63.5)
- added TP9: TestPoint, Connector_Pin:Pin_D1.3mm_L11.0mm, F.Cu at (178.7, 82.5)
- R2: value 5mOhm -> solderBridge
- TP1: value ForkTerminal -> TestPoint; footprint Connector_Pin:Pin_D1.1mm_L8.5mm_W2.5mm_FlatFork -> Connector_Pin:Pin_D1.3mm_L11.0mm
- TP3: footprint Connector_Pin:Pin_D1.3mm_L11.0mm -> Connector_Pin:Pin_D1.1mm_L10.2mm_W3.5mm_Flat
- moved D4 137.9 mm to (237.8, 112.3), turned to -90 degrees
- moved Q5 126.3 mm to (225.2, 63.2), turned to -90 degrees
- moved Q4 121.6 mm to (215.1, 39.5)
- moved R5 110.1 mm to (226.1, 50.2), turned to 90 degrees
- moved R2 103.7 mm to (221.5, 50.2), turned to -90 degrees
- moved Q2 102.5 mm to (209.6, 66.0), turned to 180 degrees
- moved R11 102.2 mm to (238.1, 100.8), turned to -90 degrees
- moved R12 101.2 mm to (237.8, 118.0), turned to -90 degrees
- moved SW5 101.0 mm to (216.0, 109.2)
- moved Q3 100.7 mm to (199.3, 42.3), turned to -90 degrees
- moved TP1 99.3 mm to (169.5, 44.5)
- moved TP3 97.5 mm to (161.8, 36.5)
- moved C13 97.2 mm to (232.3, 51.6), turned to 90 degrees
- moved C4 93.0 mm to (229.7, 51.6), turned to 90 degrees
- moved C9 92.2 mm to (197.7, 56.5)
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Connections:
- C12 pad 2: Net-(Q4-D) -> Net-(Q5-S)
- C14 pad 1: Net-(Q5-D) -> /Vout
- C15 pad 1: Net-(Q5-D) -> /Vout
- Q5 pad 3: Net-(Q4-D) -> Net-(Q5-S)
- R16 pad 1: Net-(Q5-D) -> /Vout
- R18 pad 1: VDD -> GNDS
- R18 pad 2: Net-(U1A-MODE1) -> Net-(U1A-SYNC/SPRD)
- R2 pad 1: unconnected-(R2-Pad1) -> Net-(Q4-D)
- R2 pad 2: unconnected-(R2-Pad2) -> Net-(Q5-S)
- R5 pad 2: Net-(Q5-D) -> /Vout
- R9 pad 1: Net-(Q5-D) -> /Vout
- SW2 pad 1: Net-(U1A-MODE2) -> GNDS
- SW2 pad 2: Net-(U1A-MODE1) -> GNDS
- SW2 pad 3: GNDS -> Net-(R34-Pad2)
- SW2 pad 4: GNDS -> Net-(R33-Pad2)
- SW3 pad 1: Net-(SW3-Pad1) -> /manual_bus
- SW3 pad 2: Net-(SW3-Pad1) -> /manual_bus
- SW3 pad 3: Net-(SW3-Pad1) -> /manual_bus
- SW3 pad 4: Net-(SW3-Pad1) -> /manual_bus
- SW3 pad 5: Net-(SW3-Pad1) -> /manual_bus
- SW3 pad 6: Net-(SW3-Pad1) -> /manual_bus
- SW4 pad 1: Net-(SW3-Pad1) -> /manual_bus
- SW4 pad 3: Net-(SW3-Pad1) -> /manual_bus
- TP1 pad 1: unconnected-(TP1-Pad1) -> GNDPWR
- U1 pad 16: Net-(Q5-D) -> /Vout
- U1 pad 2: Net-(U1A-MODE2) -> GNDS
- U1 pad 21: Net-(Q4-D) -> Net-(Q5-S)
- U1 pad 28: Net-(Q5-D) -> /Vout
- U1 pad 3: Net-(U1A-MODE1) -> GNDS
- U1 pad 39: (no net) -> GNDS
- U1 pad 4: GNDS -> Net-(U1A-SYNC/SPRD)
Routing:
- net GNDS: track 0.00 -> 133.5 mm, vias 0 -> 23
- net VDD: track 0.00 -> 110.7 mm, vias 0 -> 2
- net Net-(Q5-S): track 0.00 -> 100.0 mm, vias 0 -> 2
- net Net-(Q5-D): track 0.00 -> 92.0 mm, vias 0 -> 1
- net /Vout: track 0.00 -> 91.5 mm, vias 0 -> 4
- net Net-(Q4-G): track 0.00 -> 84.4 mm, vias 0 -> 2
- net Net-(L1-Pad2): track 0.00 -> 74.6 mm, vias 0 -> 2
- net Net-(Q3-G): track 0.00 -> 73.3 mm, vias 0 -> 2
- net /PWGD: track 0.00 -> 68.6 mm, vias 0 -> 2
- net Net-(U1A-IMON): track 0.00 -> 62.8 mm, vias 0 -> 2
- net Net-(Q2-S): track 0.00 -> 53.6 mm, vias 0 -> 2
- net Net-(D2-A): track 0.00 -> 52.7 mm, vias 0 -> 1
- net Net-(Q5-G): track 0.00 -> 50.3 mm, vias 0 -> 2
- net Net-(U1A-SS): track 0.00 -> 50.3 mm, vias 0 -> 2
- net /Vin: track 0.00 -> 43.3 mm
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- added copper zone on F.Cu, net /Vin
- added copper zone on F.Cu, net /Vout
- added copper zone on B.Cu, net GNDPWR
- added copper zone on F.Cu, net GNDPWR
- added copper zone on In1.Cu, net GNDPWR
- added copper zone on In2.Cu, net GNDPWR
- added copper zone on B.Cu, net GNDS
- added copper zone on In1.Cu, net GNDS
- added copper zone on In2.Cu, net GNDS
- added copper zone on F.Cu, net Net-(L1-Pad2)
- added copper zone on F.Cu, net Net-(Q1-D)
- added copper zone on F.Cu, net Net-(Q2-S)
- added copper zone on F.Cu, net Net-(Q4-D)
- added copper zone on F.Cu, net Net-(Q5-D)
- added copper zone on F.Cu, net Net-(Q5-S)
- added copper zone on B.Cu, net VDD
Other:
- board outline added: 91.5 x 100 mm
- copper layers 2 -> 4

Commit message: semi final design and pcb layout
Parts:
- removed Q1, Q2, Q3, Q4, Q5: IPB048N15N5LF, PCM_Package_TO_SOT_SMD_AKL:TO-263-2
- removed R27: 6.8MR, PCM_Resistor_SMD_AKL:R_0805_2012Metric_Pad1.20x1.40mm_HandSolder
- removed R28: 3.3MR, PCM_Resistor_SMD_AKL:R_0805_2012Metric_Pad1.20x1.40mm_HandSolder
- removed R29: 330k, PCM_Resistor_SMD_AKL:R_0805_2012Metric_Pad1.20x1.40mm_HandSolder
- removed R30: 160k, PCM_Resistor_SMD_AKL:R_0805_2012Metric_Pad1.20x1.40mm_HandSolder
- removed R31: 82k, PCM_Resistor_SMD_AKL:R_0805_2012Metric_Pad1.20x1.40mm_HandSolder
- removed R32: 33k, PCM_Resistor_SMD_AKL:R_0805_2012Metric_Pad1.20x1.40mm_HandSolder
- removed R34: 10k, PCM_Resistor_SMD_AKL:R_0805_2012Metric_Pad1.20x1.40mm_HandSolder
- removed SW5: DIP6, Button_Switch_SMD:6DIPCFS
- removed TP10, TP11, TP12, TP13, TP14, TP15, TP16, TP18, TP19, TP2, TP9: TestPoint, Connector_Pin:Pin_D1.3mm_L11.0mm
- added C27: 220pF, PCM_Capacitor_SMD_AKL:C_0805_2012Metric, B.Cu at (76.2, 91.3)
- added H1: MountingHole_Pad, MountingHole:MountingHole_3.2mm_M3_ISO14580_Pad, F.Cu at (30.0, 90.2)
- added H2: MountingHole_Pad, MountingHole:MountingHole_3.2mm_M3_ISO14580_Pad, F.Cu at (30.0, 44.2)
- added H3: MountingHole_Pad, MountingHole:MountingHole_3.2mm_M3_ISO14580_Pad, F.Cu at (118.0, 44.2)
- added H4: MountingHole_Pad, MountingHole:MountingHole_3.2mm_M3_ISO14580_Pad, F.Cu at (118.0, 90.2)
- added Q10: IRFB4615, PCM_Package_TO_SOT_THT_AKL:TO-220-3_Vertical_GDS, F.Cu at (61.4, 44.0)
- added Q11: IRFB4615, PCM_Package_TO_SOT_THT_AKL:TO-220-3_Vertical_GDS, F.Cu at (88.0, 48.5)
- added Q7: IRFB4615, PCM_Package_TO_SOT_THT_AKL:TO-220-3_Vertical_GDS, F.Cu at (65.5, 49.9)
- added Q8: IRFB4615, PCM_Package_TO_SOT_THT_AKL:TO-220-3_Vertical_GDS, F.Cu at (38.1, 47.8)
- added Q9: IRFB4615, PCM_Package_TO_SOT_THT_AKL:TO-220-3_Vertical_GDS, F.Cu at (62.0, 67.8)
- added R35: 10k, PCM_Resistor_SMD_AKL:R_0805_2012Metric_Pad1.20x1.40mm_HandSolder, B.Cu at (59.0, 79.7)
- added R36: 10k, PCM_Resistor_SMD_AKL:R_0805_2012Metric_Pad1.20x1.40mm_HandSolder, B.Cu at (61.5, 79.7)
- C1, C10, C11, C12, C16, C17, C18, C19, C20, C21, C22, C23, C24, R10, R13, R14, R15, R18, R6, R7, R8, R9: moved to B.Cu
- R16: value 100k -> 10k
- R17: value 24k -> 2.4k; moved to B.Cu
- R20: value 12k -> 1.2k; moved to B.Cu
- R21: value 9.1k -> 910R; moved to B.Cu
- R22: value 7.5k -> 750R; moved to B.Cu
- R23: value 5.1k -> 510R; moved to B.Cu
- R24: value 4.3k -> 430R; moved to B.Cu
- R25: value 15k -> 1.5k; moved to B.Cu
- R26: value 6.8k -> 680R
- R33: value 10k -> 33k; moved to B.Cu
- moved D4 193.0 mm to (46.3, 87.9)
- moved Q6 192.9 mm to (46.6, 85.4)
- moved R12 192.1 mm to (47.4, 92.8), turned to 0 degrees
- moved R11 191.8 mm to (47.6, 78.1), turned to 180 degrees
- moved C13 152.5 mm to (80.2, 62.3), turned to -90 degrees
- moved C4 147.3 mm to (82.8, 62.2), turned to -90 degrees
- moved R2 141.4 mm to (80.2, 43.0), turned to 0 degrees
- moved C9 139.2 mm to (58.5, 57.1), turned to -90 degrees
- moved R5 138.0 mm to (88.2, 56.8), turned to 0 degrees
- moved C26 136.3 mm to (97.2, 59.0), turned to -90 degrees
- moved C8 135.7 mm to (62.0, 57.1), turned to -90 degrees
- moved L1 134.8 mm to (77.5, 52.8)
- moved TP3 134.5 mm to (28.5, 55.0)
- moved TP4 134.4 mm to (28.5, 62.0)
- moved TP7 134.3 mm to (36.5, 55.0)
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Connections:
- net Net-(D2-A) renamed /GateVcc
- net Net-(D2-K) renamed /BST1
- net Net-(D3-K) renamed /BST2
- net Net-(Q1-D) renamed /VinP
- net Net-(Q2-S) renamed /SW1
- net Net-(Q5-S) renamed /SW2
- net Net-(U1A-FB1) renamed /FB1
- net Net-(U1A-FB2) renamed /FB2
- net Net-(U1A-SNSN1) renamed /SNSN1
- net Net-(U1A-SNSN2) renamed /SNSN2
- net Net-(U1A-SNSP1) renamed /SNSP1
- net Net-(U1A-SNSP2) renamed /SNSP2
- net Net-(U1A-SS) renamed /SS
- net Net-(U1A-VC1) renamed /VC1
- net Net-(U1A-VC2) renamed /VC2
- R33 pad 1: VDD -> /IMON
- R33 pad 2: Net-(R33-Pad2) -> GNDS
- SW2 pad 1: GNDS -> /MODE1
- SW2 pad 2: GNDS -> /MODE2
- SW2 pad 3: Net-(R34-Pad2) -> VDD
- SW2 pad 4: Net-(R33-Pad2) -> VDD
- U1 pad 10: Net-(U1A-IMON) -> /IMON
- U1 pad 2: GNDS -> /MODE2
- U1 pad 20: Net-(Q5-G) -> /TG2
- U1 pad 24: Net-(Q4-G) -> /BG2
- U1 pad 26: Net-(Q3-G) -> /BG1
- U1 pad 3: GNDS -> /MODE1
- U1 pad 32: Net-(Q2-G) -> /TG1
- U1 pad 37: Net-(Q1-G) -> /DG
Routing:
- net GNDS: track 133.5 -> 37.2 mm, vias 23 -> 62
- net Net-(Q4-G): track 84.4 -> 0.00 mm, vias 2 -> 0
- net Net-(Q11-D): track 92.0 -> 16.1 mm
- net Net-(Q3-G): track 73.3 -> 0.00 mm, vias 2 -> 0
- net VDD: track 110.7 -> 39.0 mm
- net Net-(L1-Pad2): track 74.6 -> 5.93 mm, vias 2 -> 1
- net Net-(U1A-IMON): track 62.8 -> 0.00 mm, vias 2 -> 0
- net /SW2: track 100.0 -> 41.1 mm
- net /DG: track 0.00 -> 53.5 mm
- net Net-(Q5-G): track 50.3 -> 0.00 mm, vias 2 -> 0
- net /SS: track 50.3 -> 6.83 mm, vias 2 -> 1
- net /SW1: track 53.6 -> 11.5 mm, vias 2 -> 3
- net Net-(Q1-G): track 42.1 -> 0.00 mm
- net /BG2: track 0.00 -> 38.2 mm
- net Net-(Q2-G): track 34.8 -> 0.00 mm, vias 2 -> 0
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- added copper zone on In2.Cu, net /Vout
- added copper zone on F.Cu, net GNDS
- removed copper zone on B.Cu, net VDD
Other:
- board size 91.5 x 100 mm -> 98 x 56 mm
- board text added: "+"
- board text added: "-"
- board text added: "1"
- board text added: "12V"
- board text added: "15V"
- board text added: "2"
- board text added: "20V"
- board text added: "24V"
- board text added: "5V"
- board text added: "9V"
- board text added: "By Thomas Vosters and Stan Coene"
- board text added: "For Group T Course 'Power Electronics'"
- board text added: "IN"
- board text added: "LT8210 Development Board"
- board text added: "MODE"
- board text added: "Power ground"
- board text added: "SPRD"
- board text added: "Voltage setting"
- board text added: "With Adjustable Output Voltage"
- board text added: "ground"
- board text added: "out"
- board text added: "signal"

Commit message: added local libraries
Parts:
- C1, C10, C11, C12, C16, C17, C18, C19, C20, C21, C22, C23, C24, C25, C26, C27: footprint PCM_Capacitor_SMD_AKL:C_0805_2012Metric -> buckFootprints:C_0805_2012Metric
- C13, C4: footprint Capacitor_SMD:C_1206_3216Metric_Pad1.33x1.80mm_HandSolder -> buckFootprints:C_1206_3216Metric_Pad1.33x1.80mm_HandSolder
- C14, C15: footprint PCM_Capacitor_THT_AKL:CP_Radial_D10.0mm_P5.00mm -> buckFootprints:CP_Radial_D10.0mm_P5.00mm
- C5, C7: footprint PCM_Capacitor_THT_AKL:CP_Radial_D16.0mm_P7.50mm -> buckFootprints:CP_Radial_D16.0mm_P7.50mm
- C8, C9: footprint Capacitor_SMD:C_1210_3225Metric_Pad1.33x2.70mm_HandSolder -> buckFootprints:C_1210_3225Metric_Pad1.33x2.70mm_HandSolder
- D2, D3: footprint PCM_Diode_SMD_AKL:D_SMB -> buckFootprints:D_SMB
- D4: footprint PCM_LED_THT_AKL_Double:LED_D3.0mm -> buckFootprints:LED_D3.0mm
- H1, H2, H3, H4: footprint MountingHole:MountingHole_3.2mm_M3_ISO14580_Pad -> buckFootprints:MountingHole_3.2mm_M3_ISO14580_Pad
- L1: footprint Inductor_SMD_Wurth:IND_1210-WE-HCC_WRE -> buckFootprints:IND_1210-WE-HCC_WRE
- Q10, Q11, Q7, Q8, Q9: footprint PCM_Package_TO_SOT_THT_AKL:TO-220-3_Vertical_GDS -> buckFootprints:TO-220-3_Vertical_GDS
- Q6: footprint PCM_Package_TO_SOT_THT_AKL:TO-92_Inline_Wide_CBE -> buckFootprints:TO-92_Inline_Wide_CBE
- R1, R2, R5: footprint PCM_Resistor_SMD_AKL:R_2512_6332Metric -> buckFootprints:R_2512_6332Metric
- R10, R11, R12, R13, R14, R15, R16, R17, R18, R20, R21, R22, R23, R24, R25, R26, R33, R35, R36, R6, R7, R8, R9: footprint PCM_Resistor_SMD_AKL:R_0805_2012Metric_Pad1.20x1.40mm_HandSolder -> buckFootprints:R_0805_2012Metric_Pad1.20x1.40mm_HandSolder
- SW2, SW6: footprint Button_Switch_SMD:2DIPCFS -> buckFootprints:2DIPCFS
- SW3: footprint Button_Switch_SMD:6DIPCFS -> buckFootprints:6DIPCFS
- SW4: footprint Button_Switch_SMD:SW6_76SD01ST_GHL -> buckFootprints:SW6_76SD01ST_GHL
- TP1, TP21, TP7, TP8: footprint Connector_Pin:Pin_D1.3mm_L11.0mm -> buckFootprints:Pin_D1.3mm_L11.0mm
- TP3, TP4, TP5, TP6: footprint Connector_Pin:Pin_D1.1mm_L10.2mm_W3.5mm_Flat -> buckFootprints:Pin_D1.1mm_L10.2mm_W3.5mm_Flat
- U1: footprint Converter_DCDC:05-08-1772_ADI-M -> buckFootprints:05-08-1772_ADI-M
