File: adjustableBuck.kicad_sch (KiCad schematic)
At the start: 77 parts, among them Q1 IPB048N15N5LF, Q2 IPB048N15N5LF, Q3 IPB048N15N5LF, Q4 IPB048N15N5LF, Q5 IPB048N15N5LF, Q6 BC547, SW1 DIP6, SW2 DIP2, SW3 DIP6, SW4 76SD01ST, SW5 DIP6, U1 LT8210EFE

Commit message: First board layout
Parts:
- removed C2: 470uF 35V, PCM_Capacitor_THT_AKL:CP_Radial_D10.0mm_P5.00mm, symbol PCM_Capacitor_AKL:CP_Radial_D10.0mm_P5.00mm
- removed C3: 10uF 100V, Capacitor_SMD:C_1210_3225Metric_Pad1.33x2.70mm_HandSolder, symbol PCM_Capacitor_AKL:C_1210
- removed C6: C_0805, PCM_Capacitor_SMD_AKL:C_0805_2012Metric, symbol PCM_Capacitor_AKL:C_0805
- removed D1: MURS160, PCM_Diode_SMD_AKL:D_SMB, symbol PCM_Diode_AKL:MURS160
- removed R3, R4: R_0805, PCM_Resistor_SMD_AKL:R_0805_2012Metric_Pad1.20x1.40mm_HandSolder, symbol PCM_Resistor_AKL:R_0805
- removed SW1: DIP6, Button_Switch_SMD:6DIPCFS, symbol Switch:SW_DIP_x06
- added R18: 10k, PCM_Resistor_SMD_AKL:R_0805_2012Metric_Pad1.20x1.40mm_HandSolder, symbol PCM_Resistor_AKL:R_0805
- added SW6: DIP2, Button_Switch_SMD:2DIPCFS, symbol Switch:SW_DIP_x02
- added TP10, TP11, TP12, TP13, TP14, TP15, TP16, TP18, TP19, TP2, TP20, TP21, TP7, TP8, TP9: TestPoint, Connector_Pin:Pin_D1.3mm_L11.0mm, symbol Connector:TestPoint
- added TP4, TP5, TP6: ProbePoint, Connector_Pin:Pin_D1.1mm_L10.2mm_W3.5mm_Flat, symbol Connector:TestPoint_Alt
- R2: value 5mOhm -> solderBridge
- TP1: value ForkTerminal -> TestPoint; footprint Connector_Pin:Pin_D1.1mm_L8.5mm_W2.5mm_FlatFork -> Connector_Pin:Pin_D1.3mm_L11.0mm
- TP3: footprint Connector_Pin:Pin_D1.3mm_L11.0mm -> Connector_Pin:Pin_D1.1mm_L10.2mm_W3.5mm_Flat
Connections:
- net GNDPWR: now also TP1.1, TP21.1, TP4.1, TP6.1
- net GNDS: now also U1.39 (SGND), R18.1, TP2.1; no longer U1.4 (SYNC/SPRD)
- net VDD: now also SW6.3, TP9.1
- net Vin: now also TP7.1
- net manual_bus: now also SW3.1, SW3.2, SW3.3, SW3.4, SW3.5, SW3.6, SW4.1, SW4.3
- net Vout: now reaches C14.1, C15.1, C25.1, C26.1, R16.1, R5.2, R9.1, U1.16 (VOUT), U1.28 (ExtVcc)
- net Vout: now also TP20.1, TP5.1, TP8.1; no longer C13.1, C4.1, Q5.2 (D), R5.1, R8.1
- net at C24.2, SW5.1, SW5.2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: now also TP13.1
- net at C23.2, R15.2, U1.12 (VC2): now also TP15.1
- net at C12.2, Q5.3 (S), U1.21 (SW2): now also R2.2, TP12.1; no longer L1.1, Q4.2 (D)
- net at L1.2, R1.2, R7.1: now also TP18.1
- net at C11.1, D2.2 (A), D3.2 (A)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: now also TP10.1
- net at C18.2, R14.2, U1.11 (VC1): now also TP14.1
- net at C10.2, Q2.3 (S), Q3.2 (D)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: now also TP11.1
- net at R2.1: now also L1.1, Q4.2 (D)
- net at C17.2, U1.9 (SS): now also TP16.1
- new net: C13.1, C4.1, Q5.2 (D), R5.1, R8.1, TP19.1
- new net: R18.2, SW6.2, U1.4 (SYNC/SPRD)
Other:
- note added: "Power Good? LED"
- note added: "fsw = 257kHz"
- moved on the sheet: R33, R34, SW2

Commit message: semi final design and pcb layout
Parts:
- removed Q1, Q2, Q3, Q4, Q5: IPB048N15N5LF, PCM_Package_TO_SOT_SMD_AKL:TO-263-2, symbol PCM_Transistor_MOSFET_AKL:IPB048N15N5LF
- removed R34: 10k, PCM_Resistor_SMD_AKL:R_0805_2012Metric_Pad1.20x1.40mm_HandSolder, symbol PCM_Resistor_AKL:R_0805
- removed TP20: TestPoint, Connector_Pin:Pin_D1.3mm_L11.0mm, symbol Connector:TestPoint
- added C27: 220pF, PCM_Capacitor_SMD_AKL:C_0805_2012Metric, symbol PCM_Capacitor_AKL:C_0805
- added H1, H2, H3, H4: MountingHole_Pad, MountingHole:MountingHole_3.2mm_M3_ISO14580_Pad, symbol Mechanical:MountingHole_Pad
- added Q10, Q11, Q7, Q8, Q9: IRFB4615, PCM_Package_TO_SOT_THT_AKL:TO-220-3_Vertical_GDS, symbol PCM_Transistor_MOSFET_AKL:IRFB4615
- added R35, R36: 10k, PCM_Resistor_SMD_AKL:R_0805_2012Metric_Pad1.20x1.40mm_HandSolder, symbol PCM_Resistor_AKL:R_0805
- C24, R27, R28, R29, R30, R31, R32, SW5: now not fitted
- R16: value 100k -> 10k
- R17: value 24k -> 2.4k
- R20: value 12k -> 1.2k
- R21: value 9.1k -> 910R
- R22: value 7.5k -> 750R
- R23: value 5.1k -> 510R
- R24: value 4.3k -> 430R
- R25: value 15k -> 1.5k
- R26: value 6.8k -> 680R
- R33: value 10k -> 33k
Connections:
- net GNDPWR: now also H1.1, H2.1, H3.1, H4.1, Q10.3 (S), Q9.3 (S)
- net GNDS: now also R33.2, C27.2, R35.2, R36.2; no longer SW2.1, SW2.2, U1.2 (MODE2), U1.3 (MODE1)
- net VDD: now also SW2.3, SW2.4; no longer R33.1
- net Vin: now also Q8.3 (S)
- net SW2: now reaches C12.2, R2.2, TP12.1, U1.21 (SW2)
- net SW2: now also Q11.3 (S)
- net VC1: now reaches C18.2, R14.2, TP14.1, U1.11 (VC1)
- net at C13.1, C4.1, R5.1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: now also Q11.2 (D)
- net at C24.2, SW5.1, SW5.2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: no longer TP13.1, U1.10 (IMON)
- net VC2: now reaches C23.2, R15.2, TP15.1, U1.12 (VC2)
- net SW1: now reaches C10.2, R1.1, R6.2, TP11.1, U1.31 (SW1)
- net SW1: now also Q7.3 (S), Q9.2 (D)
- net at L1.1, R2.1: now also Q10.2 (D)
- net SS: now reaches C17.2, TP16.1, U1.9 (SS)
- net GateVcc: now reaches C11.1, D2.2 (A), D3.2 (A), TP10.1, U1.27 (GateVcc)
- net SNSP2: now reaches C22.1, R8.2, U1.19 (SNSP2)
- net BST2: now reaches C12.1, D3.1 (K), U1.22 (BST2)
- net BG1: now reaches U1.26 (BG1)
- net BG1: now also Q9.1 (G)
- net SNSP1: now reaches C21.1, R6.1, U1.34 (SNSP1)
- net SNSN1: now reaches C21.2, R7.2, U1.33 (SNSN1)
- net TG2: now reaches U1.20 (TG2)
- net TG2: now also Q11.1 (G)
- net VinP: now reaches C5.1, C7.1, C8.1, C9.1, U1.36 (VinP)
- net VinP: now also Q7.2 (D), Q8.2 (D)
- net SNSN2: now reaches C22.2, R9.2, U1.18 (SNSN2)
- net BG2: now reaches U1.24 (BG2)
- net BG2: now also Q10.1 (G)
- net FB2: now reaches SW4.5, U1.13 (FB2)
- net FB1: now reaches SW4.2, U1.14 (FB1)
- net BST1: now reaches C10.1, D2.1 (K), U1.30 (BST1)
- net TG1: now reaches U1.32 (TG1)
- net TG1: now also Q7.1 (G)
- net DG: now reaches U1.37 (DG)
- net DG: now also Q8.1 (G)
- new net IMON: C27.1, R33.1, TP13.1, U1.10 (IMON)
- new net MODE1: R35.1, SW2.1, U1.3 (MODE1)
- new net MODE2: R36.1, SW2.2, U1.2 (MODE2)
- no-connect marks 0 -> 2
Other:
- moved on the sheet: C11, SW2

Commit message: added local libraries
Parts:
- C1, C10, C11, C12, C16, C17, C18, C19, C20, C21, C22, C23, C24, C25, C26, C27: symbol PCM_Capacitor_AKL:C_0805 -> bucklibrary:C_0805
- C13, C4: symbol PCM_Capacitor_AKL:C_1206 -> bucklibrary:C_1206
- C14, C15: symbol PCM_Capacitor_AKL:CP_Radial_D10.0mm_P5.00mm -> bucklibrary:CP_Radial_D10.0mm_P5.00mm
- C5, C7: symbol PCM_Capacitor_AKL:CP_Radial_D16.0mm_P7.50mm -> bucklibrary:CP_Radial_D16.0mm_P7.50mm
- C8, C9: symbol PCM_Capacitor_AKL:C_1210 -> bucklibrary:C_1210
- D2, D3: symbol PCM_Diode_AKL:MURS160 -> bucklibrary:MURS160
- D4: symbol Device:LED -> bucklibrary:LED
- H1, H2, H3, H4: symbol Mechanical:MountingHole_Pad -> bucklibrary:MountingHole_Pad
- L1: symbol Transformer:7443320680 -> bucklibrary:7443320680
- Q10, Q11, Q7, Q8, Q9: symbol PCM_Transistor_MOSFET_AKL:IRFB4615 -> bucklibrary:IRFB4615
- Q6: symbol PCM_Transistor_BJT_AKL:BC547 -> bucklibrary:BC547
- R1, R2, R5: symbol PCM_Resistor_AKL:R_2512 -> bucklibrary:R_2512
- R10, R11, R12, R13, R14, R15, R16, R17, R18, R20, R21, R22, R23, R24, R25, R26, R27, R28, R29, R30, R31, R32, R33, R35, R36, R6, R7, R8, R9: symbol PCM_Resistor_AKL:R_0805 -> bucklibrary:R_0805
- SW2, SW6: symbol Switch:SW_DIP_x02 -> bucklibrary:SW_DIP_x02
- SW3, SW5: symbol Switch:SW_DIP_x06 -> bucklibrary:SW_DIP_x06
- SW4: symbol Switch:76SD01ST -> bucklibrary:76SD01ST
- TP1, TP10, TP11, TP12, TP13, TP14, TP15, TP16, TP18, TP19, TP2, TP21, TP7, TP8, TP9: symbol Connector:TestPoint -> bucklibrary:TestPoint
- TP3, TP4, TP5, TP6: symbol Connector:TestPoint_Alt -> bucklibrary:TestPoint_Alt
- U1: symbol Converter_DCDC:LT8210EFE -> bucklibrary:LT8210EFE
